File: KiCAD/ItsyBitsy_PanelMount_VerticalAdapter/ItsyBitsy_PanelMount_VerticalAdapter.kicad_pcb (KiCad board)
At the start: 2 copper layers, 35.6 x 40.6 mm, 5 parts, among them J1 Conn_01x14_Socket, J2 Conn_01x14_Socket, J3 Conn_01x14_Socket, J4 Conn_01x14_Socket, J5 Conn_02x14_Odd_Even

Commit message: added copper fills to every module, to maybe possibly increase structural rigidity.
Routing:
- added copper zone on B.Cu, net (none)
- added copper zone on F.Cu, net (none)
Changed lines of the file:
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@@
 		(net 28)
 	)
+	(zone
+		(net 0)
+		(net_name "")
+		(layers "F&B.Cu")
+		(hatch edge 0.5)
+		(connect_pads
+			(clearance 0.5)
+		)
+		(min_thickness 0.25)
+		(filled_areas_thickness no)
+		(fill yes
+			(thermal_gap 0.5)
+			(thermal_bridge_width 0.5)
+			(island_removal_mode 1)
+			(island_area_min 10)
+		)
+		(polygon
+			(pts
+				(xy 0 0) (xy 35.56 0) (xy 35.56 5.08) (xy 30.48 40.64) (xy 7.62 40.64) (xy 0 5.08)
+			)
+		)
+	)
 )

Commit message: added PCBWay print identification silkscreen text to each component
Other:
- board text added: "WayWayWay"
Changed lines of the file:
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@@
 		(layer "Edge.Cuts")
+	)
+	(gr_text "WayWayWay"
+		(at 6.5 25.25 -90)
+		(layer "B.SilkS")
+		(effects
+			(font
+				(size 1 1)
+				(thickness 0.15)
+			)
+			(justify left top mirror)
+		)
 	)
 	(gr_text "ItsyBitsy Panel-Mount\nVertical Adapter\nV1\nMostlyCoraGrace"
