File: KiCAD/ToggleSwitch_1U7HP1x_A/ToggleSwitch_1U7HP1x_A.kicad_pcb (KiCad board)
At the start: 2 copper layers, 35.3 x 39.7 mm, 7 parts, among them SW1 SW_SPST_M6_MOUNT

Commit message: toggle switch v2 updates
Routing:
- added copper zone on B.Cu, net (none)
- added copper zone on F.Cu, net (none)
Other:
- board text added: "WayWayWay"
Changed lines of the file:
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@@
 		(property "Reference" "H3"
 			(at 5.84 -0.05 0)
-			(layer "F.SilkS")
-			(effects
-				(font
-					(size 1 1)
-					(thickness 0.15)
-				)
-				(justify right)
+			(layer "B.SilkS")
+			(effects
+				(font
+					(size 1 1)
+					(thickness 0.15)
+				)
+				(justify left mirror)
 			)
 		)
@@
 		(fp_circle
 			(center 0 0)
+			(end 2.84 0)
+			(stroke
+				(width 0.1)
+				(type solid)
+			)
+			(fill no)
+			(layer "Dwgs.User")
+		)
+		(fp_circle
+			(center 0 0)
+			(end 3.45 0)
+			(stroke
+				(width 0.05)
+				(type solid)
+			)
+			(fill no)
+			(layer "Dwgs.User")
+		)
+		(fp_circle
+			(center 0 0)
 			(end 3.2 0)
 			(stroke
@@
 			(fill no)
 			(layer "Cmts.User")
-		)
-		(fp_circle
-			(center 0 0)
-			(end 3.45 0)
-			(stroke
-				(width 0.05)
-				(type solid)
-			)
-			(fill no)
-			(layer "F.CrtYd")
 		)
 		(fp_text user "${REFERENCE}"
@@
 		(pad "" np_thru_hole oval
 			(at 0 0)
-			(size 4.8 3.2)
-			(drill oval 4.8 3.2)
+			(size 4.34 3.2)
+			(drill oval 4.34 3.2)
 			(layers "*.Cu" "*.Mask")
 		)
@@
 		(at 28.62 14.95)
 		(property "Reference" "D1"
-			(at 0 -5 0)
-			(unlocked yes)
-			(layer "F.SilkS")
-			(effects
-				(font
-					(size 1 1)
-					(thickness 0.1)
-				)
+			(at 0 5.55 0)
+			(unlocked yes)
+			(layer "B.SilkS")
+			(effects
+				(font
+					(size 1 1)
+					(thickness 0.125)
+				)
+				(justify mirror)
 			)
 		)
@@
 		)
 		(fp_text user "${REFERENCE}"
-			(at 0 5 0)
+			(at 0 5.55 0)
 			(unlocked yes)
 			(layer "F.Fab")
@@
 		(property "Reference" "H4"
 			(at -3.683 0 0)
-			(layer "F.SilkS")
-			(effects
-				(font
-					(size 1 1)
-					(thickness 0.15)
-				)
-				(justify right)
+			(layer "B.SilkS")
+			(effects
+				(font
+					(size 1 1)
+					(thickness 0.15)
+				)
+				(justify left mirror)
 			)
 		)
@@
 		(fp_circle
 			(center 0 0)
+			(end 2.84 0)
+			(stroke
+				(width 0.1)
+				(type solid)
+			)
+			(fill no)
+			(layer "Dwgs.User")
+		)
+		(fp_circle
+			(center 0 0)
+			(end 3.45 0)
+			(stroke
+				(width 0.05)
+				(type solid)
+			)
+			(fill no)
+			(layer "Dwgs.User")
+		)
+		(fp_circle
+			(center 0 0)
 			(end 3.2 0)
 			(stroke
@@
 			(fill no)
 			(layer "Cmts.User")
-		)
-		(fp_circle
-			(center 0 0)
-			(end 3.45 0)
-			(stroke
-				(width 0.05)
-				(type solid)
-			)
-			(fill no)
-			(layer "F.CrtYd")
 		)
 		(fp_text user "${REFERENCE}"
@@
 		(pad "" np_thru_hole oval
 			(at 0 0)
-			(size 4.8 3.2)
-			(drill oval 4.8 3.2)
+			(size 4.34 3.2)
+			(drill oval 4.34 3.2)
 			(layers "*.Cu" "*.Mask")
 		)
@@
 			(at 0 4.15 0)
 			(unlocked yes)
-			(layer "F.SilkS")
+			(layer "B.SilkS")
 			(effects
 				(font
@@
 					(thickness 0.1)
 				)
+				(justify mirror)
 			)
 		)
@@
 		(property "Reference" "H2"
 			(at 5.84 0 0)
-			(layer "F.SilkS")
-			(effects
-				(font
-					(size 1 1)
-					(thickness 0.15)
-				)
-				(justify right)
+			(layer "B.SilkS")
+			(effects
+				(font
+					(size 1 1)
+					(thickness 0.15)
+				)
+				(justify left mirror)
 			)
 		)
@@
 		(fp_circle
 			(center 0 0)
+			(end 2.84 0)
+			(stroke
+				(width 0.1)
+				(type solid)
+			)
+			(fill no)
+			(layer "Dwgs.User")
+		)
+		(fp_circle
+			(center 0 0)
+			(end 3.45 0)
+			(stroke
+				(width 0.05)
+				(type solid)
+			)
+			(fill no)
+			(layer "Dwgs.User")
+		)
+		(fp_circle
+			(center 0 0)
 			(end 3.2 0)
 			(stroke
@@
 			(fill no)
 			(layer "Cmts.User")
-		)
-		(fp_circle
-			(center 0 0)
-			(end 3.45 0)
-			(stroke
-				(width 0.05)
-				(type solid)
-			)
-			(fill no)
-			(layer "F.CrtYd")
 		)
 		(fp_text user "${REFERENCE}"
@@
 		(pad "" np_thru_hole oval
 			(at 0 0)
-			(size 4.8 3.2)
-			(drill oval 4.8 3.2)
+			(size 4.34 3.2)
+			(drill oval 4.34 3.2)
 			(layers "*.Cu" "*.Mask")
 		)
@@
 			(at -0.25 -8.225 0)
 			(unlocked yes)
-			(layer "F.SilkS")
+			(layer "B.SilkS")
 			(effects
 				(font
@@
 					(thickness 0.1)
 				)
+				(justify mirror)
 			)
 		)
@@
 		(property "Reference" "H5"
 			(at -3.683 0 0)
-			(layer "F.SilkS")
-			(effects
-				(font
-					(size 1 1)
-					(thickness 0.15)
-				)
-				(justify right)
+			(layer "B.SilkS")
+			(effects
+				(font
+					(size 1 1)
+					(thickness 0.15)
+				)
+				(justify left mirror)
 			)
 		)
@@
 		(fp_circle
 			(center 0 0)
+			(end 2.84 0)
+			(stroke
+				(width 0.1)
+				(type solid)
+			)
+			(fill no)
+			(layer "Dwgs.User")
+		)
+		(fp_circle
+			(center 0 0)
+			(end 3.45 0)
+			(stroke
+				(width 0.05)
+				(type solid)
+			)
+			(fill no)
+			(layer "Dwgs.User")
+		)
+		(fp_circle
+			(center 0 0)
 			(end 3.2 0)
 			(stroke
@@
 			(fill no)
 			(layer "Cmts.User")
-		)
-		(fp_circle
-			(center 0 0)
-			(end 3.45 0)
-			(stroke
-				(width 0.05)
-				(type solid)
-			)
-			(fill no)
-			(layer "F.CrtYd")
 		)
 		(fp_text user "${REFERENCE}"
@@
 		(pad "" np_thru_hole oval
 			(at 0 0)
-			(size 4.8 3.2)
-			(drill oval 4.8 3.2)
+			(size 4.34 3.2)
+			(drill oval 4.34 3.2)
 			(layers "*.Cu" "*.Mask")
 		)
@@
 		(layer "Edge.Cuts")
 	)
+	(gr_text "WayWayWay"
+		(at 6 25.5 270)
+		(layer "B.SilkS")
+		(effects
+			(font
+				(size 0.8 0.8)
+				(thickness 0.1)
+			)
+			(justify left top mirror)
+		)
+	)
 	(gr_text "ToggleSwitch\n1U7HP1X_A V2\nMostlyCoraGrace"
-		(at 7.3 17 270)
-		(layer "F.SilkS")
+		(at 7.5 28.5 270)
+		(layer "B.SilkS")
 		(effects
 			(font
@@
 				(thickness 0.15)
 			)
-			(justify left bottom)
-		)
-	)
+			(justify left bottom mirror)
+		)
+	)
+	(zone
+		(net 0)
+		(net_name "")
+		(layer "F.Cu")
+		(name "Filled.Front")
+		(hatch edge 0.5)
+		(connect_pads
+			(clearance 0.5)
+		)
+		(min_thickness 0.25)
+		(filled_areas_thickness no)
+		(fill yes
+			(thermal_gap 0.5)
+			(thermal_bridge_width 0.5)
+			(island_removal_mode 1)
+			(island_area_min 10)
+		)
+		(polygon
+			(pts
+				(xy 0 2.5) (xy 35 2.5) (xy 35 42) (xy 0 42)
+			)
+		)
+	)
+	(zone
+		(net 0)
+		(net_name "")
+		(layer "B.Cu")
+		(name "Filled.Back")
+		(hatch edge 0.5)
+		(priority 1)
+		(connect_pads
+			(clearance 0.5)
+		)
+		(min_thickness 0.25)
+		(filled_areas_thickness no)
+		(fill yes
+			(thermal_gap 0.5)
+			(thermal_bridge_width 0.5)
+			(island_removal_mode 1)
+			(island_area_min 10)
+		)
+		(polygon
+			(pts
+				(xy 0 2.5) (xy 35 2.5) (xy 35 42) (xy 0 42)
+			)
+		)
+	)

Commit message: fixed mounting hole positioning for ToggleSwitch_1U7HP1x_A
Parts:
- moved H4 1.80 mm to (27.9, 5.40)
Changed lines of the file:
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@@
 	(footprint "EXC:MountingHole_3.2mm_M3"
 		(layer "F.Cu")
-		(at 29.74 5.4)
+		(at 27.94 5.4)
 		(descr "Mounting Hole 3.2mm, no annular, M3")
 		(tags "mounting hole 3.2mm no annular m3")
