File: KiCAD/Motherboard_V2/Motherboard_V2.kicad_sch (KiCad schematic)
At the start: 1 part

Commit message: motherboard tinkering
Parts:
- added H1: Eurorack_M3_MountingHole, EXC:MountingHole_3.2mm_M3, symbol EXC:Eurorack_M3_MountingHole
- added PP1: ~, EXC:Adafruit_Perma-Proto_Mint-Tin-Size, symbol EXC:Adafruit_Perma-Proto_Mint-Tin-Size
- added TLC1, TLC2, TLC3: Adafruit_24-Channel_PWM_LED_Driver_TLC5947, EXC:Adafruit_24-Channel_PWM_LED_Driver_TLC5947, symbol EXC:Adafruit_24-Channel_PWM_LED_Driver_TLC5947
Connections:
- net LAT: now reaches GCE1.16 (D2)
- net LAT: now also TLC1.49 (LAT)
- net MOSI: now reaches GCE1.58 (D51/MOSI)
- net MOSI: now also TLC1.52 (DIN)
- net SCK: now reaches GCE1.59 (D52/SCK)
- net SCK: now also TLC1.51 (CLK)
- net GND: now reaches GCE1.80 (GND)
- net GND: now also GCE1.81 (GND), PP1.5 (GND), PP1.6 (GND), TLC1.53 (GND), TLC1.59 (GND), TLC2.53 (GND), TLC2.59 (GND), TLC3.53 (GND)
- net 5V: now reaches GCE1.82 (5V)
- net 5V: now also TLC1.54 (V+), TLC1.60 (V+), TLC2.54 (V+), TLC2.60 (V+), TLC3.54 (V+)
- net 3.3: now reaches GCE1.83 (3.3)
- net Reset: now reaches GCE1.84 (RST)
- new net: TLC2.55 (LAT), TLC3.49 (LAT)
- new net: TLC2.58 (CLK), TLC3.51 (CLK)
- new net: TLC2.57 (DOUT), TLC3.52 (DIN)
- new net: TLC1.55 (LAT), TLC2.49 (LAT)
- new net: TLC1.58 (CLK), TLC2.51 (CLK)
- new net: TLC1.57 (DOUT), TLC2.52 (DIN)
- no-connect marks 0 -> 7

Commit message: motherboard noodling
Connections:
- net 3.3: now also PP1.7 (V+), PP1.8 (V+)
- net 5V: now also TLC3.60 (V+)
- net GND: now also TLC3.59 (GND)
- net LAT: now also GCE1.60 (D53/SS); no longer GCE1.16 (D2)
- no-connect marks 7 -> 10
Changed lines of the file:
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@@
+	)
+	(no_connect
+		(at 246.38 157.48)
 	)
 	(no_connect
@@
 	)
 	(no_connect
+		(at 246.38 154.94)
+	)
+	(no_connect
 		(at 177.8 152.4)
 	)
@@
 	)
 	(no_connect
+		(at 246.38 149.86)
+	)
+	(no_connect
 		(at 91.44 152.4)
 	)
@@
 	)
 	(label "LAT"
-		(at 68.58 22.86 90)
+		(at 106.68 111.76 0)
 		(effects
 			(font
@@
 		)
 	)
+	(label "5V"
+		(at 246.38 162.56 0)
+		(effects
+			(font
+				(size 1.27 1.27)
+			)
+			(justify left bottom)
+		)
+	)
 	(label "GND"
 		(at 142.24 48.26 90)
@@
 	)
 	(label "3.3"
+		(at 139.7 48.26 90)
+		(effects
+			(font
+				(size 1.27 1.27)
+			)
+			(justify left bottom)
+		)
+	)
+	(label "3.3"
 		(at 40.64 121.92 270)
 		(effects
@@
 		)
 	)
+	(label "GND"
+		(at 246.38 160.02 0)
+		(effects
+			(font
+				(size 1.27 1.27)
+			)
+			(justify left bottom)
+		)
+	)
 	(label "SCK"
 		(at 106.68 109.22 0)
@@
 			)
 			(justify right bottom)
+		)
+	)
+	(label "3.3"
+		(at 134.62 48.26 90)
+		(effects
+			(font
+				(size 1.27 1.27)
+			)
+			(justify left bottom)
 		)
 	)
@@
 		(pin "6"
 		)
+		(pin "7"
+		)
+		(pin "8"
+		)
 		(instances
